File: shark1by3by2040.kicad_pcb (KiCad board)
At the start: 2 copper layers, 0 parts

Commit message: make 1by3, do most of work on pcb
Parts:
- added A1: USB, random-keyboard-parts:JST-SR-4, B.Cu at (173.6, 55.8)
- added C1: 100nF, Capacitor_SMD:C_0805_2012Metric, B.Cu at (177.0, 71.1)
- added C10: 100nF, Capacitor_SMD:C_0805_2012Metric, B.Cu at (175.0, 73.4)
- added C11: 1uF, Capacitor_SMD:C_0805_2012Metric, B.Cu at (172.1, 75.1)
- added C12: 1uF, Capacitor_SMD:C_0805_2012Metric, B.Cu at (168.7, 78.7)
- added C13: 100nF, Capacitor_SMD:C_0805_2012Metric, B.Cu at (187.2, 57.4)
- added C14: 10uF, Capacitor_SMD:C_0805_2012Metric, B.Cu at (162.3, 74.7)
- added C15: 10uF, Capacitor_SMD:C_0805_2012Metric, B.Cu at (162.6, 64.3)
- added C16: 27pF, Capacitor_SMD:C_0805_2012Metric, B.Cu at (177.9, 101.6)
- added C17: 27pF, Capacitor_SMD:C_0805_2012Metric, B.Cu at (171.3, 101.6)
- added C2: 100nF, Capacitor_SMD:C_0805_2012Metric, B.Cu at (169.2, 89.3)
- added C3: 100nF, Capacitor_SMD:C_0805_2012Metric, B.Cu at (181.7, 81.8)
- added C4: 100nF, Capacitor_SMD:C_0805_2012Metric, B.Cu at (180.7, 88.3)
- added C5: 100nF, Capacitor_SMD:C_0805_2012Metric, B.Cu at (169.2, 91.3)
- added C6: 100nF, Capacitor_SMD:C_0805_2012Metric, B.Cu at (167.5, 84.3)
- added C7: 100nF, Capacitor_SMD:C_0805_2012Metric, B.Cu at (167.5, 80.8)
- added D1: D_Small, Diode_SMD:D_SOD-123, B.Cu at (162.9, 115.3)
- added D2: D_Small, Diode_SMD:D_SOD-123, B.Cu at (182.0, 115.3)
- added D3: D_Small, Diode_SMD:D_SOD-123, B.Cu at (201.0, 115.3)
- added H1: Daughterboard, local:UNIFIED-DAUGHTERBOARD-C3, B.Cu at (173.6, 37.8)
- added J1: SWD, Connector_PinHeader_2.54mm:PinHeader_1x04_P2.54mm_Vertical, B.Cu at (183.6, 94.5)
- added MX1: Z, marbastlib-mx:SW_MX_HS_1u, B.Cu at (154.6, 110.6)
- added MX2: X, marbastlib-mx:SW_MX_HS_1u, B.Cu at (173.6, 110.6)
- added MX3: C, marbastlib-mx:SW_MX_HS_1u, B.Cu at (192.7, 110.6)
- added R1: 27, Resistor_SMD:R_0805_2012Metric, B.Cu at (174.8, 68.8)
- added R2: 27, Resistor_SMD:R_0805_2012Metric, B.Cu at (172.5, 68.8)
- added R3: 1k, Resistor_SMD:R_0805_2012Metric, B.Cu at (186.8, 69.6)
- added R4: 1k, Resistor_SMD:R_0805_2012Metric, B.Cu at (174.6, 92.2)
- added R5: 1k, Resistor_SMD:R_0805_2012Metric, B.Cu at (165.1, 87.2)
- added SW1: SW_USB_BOOT, local:TS-1187A, B.Cu at (181.0, 74.8)
- added SW2: SW_Reset, local:TS-1187A, B.Cu at (157.8, 89.9)
- added U1: RP2040, RP2040_minimal:RP2040-QFN-56, B.Cu at (174.6, 83.3)
- added U2: W25Q128JVS, Package_SO:SOIC-8_5.23x5.23mm_P1.27mm, B.Cu at (183.3, 63.2)
- added U3: NCP1117-3.3_SOT223, Package_TO_SOT_SMD:SOT-223-3_TabPin2, B.Cu at (159.0, 70.0)
- added Y1: ABLS-12.000MHZ-B4-T, Crystal:Crystal_SMD_HC49-SD, B.Cu at (174.6, 97.0)
Routing:
- net +3V3: track 0.00 -> 155.9 mm, vias 0 -> 7
- net row0: track 0.00 -> 89.3 mm
- net col0: track 0.00 -> 66.7 mm
- net GND: track 0.00 -> 55.3 mm, vias 0 -> 6
- net col1: track 0.00 -> 48.7 mm
- net +1V1: track 0.00 -> 44.8 mm, vias 0 -> 3
- net col2: track 0.00 -> 35.7 mm
- net Net-(U1-Pad51): track 0.00 -> 27.4 mm
- net SCLK: track 0.00 -> 26.1 mm
- net Net-(U1-Pad53): track 0.00 -> 22.5 mm
- net +5V: track 0.00 -> 21.5 mm
- net Net-(J1-Pad2): track 0.00 -> 19.1 mm, vias 0 -> 2
- net SS: track 0.00 -> 18.0 mm
- net Net-(C16-Pad2): track 0.00 -> 16.3 mm
- net Net-(U1-Pad55): track 0.00 -> 16.0 mm
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- added copper zone on B.Cu, net GND
